Commit message: make gazebo and rvis joint state linked but still not able to control the servo yet

File: tb3kai_description/urdf/turtlebot3_burger.gazebo.xacro (robot description, xacro)
@@ -29,4 +29,12 @@
     </plugin>
   </gazebo>
+  <!-- ros_control plugin for laser servo -->
+  <gazebo>
+    <plugin name="gazebo_ros_control" filename="libgazebo_ros_control.so">
+      <!--robotNamespace>/open_manipulator</robotNamespace-->
+      <controlPeriod>0.001</controlPeriod>
+      <robotSimType>gazebo_ros_control/DefaultRobotHWSim</robotSimType>
+    </plugin>
+  </gazebo>
   <gazebo reference="base_link">
     <material>Gazebo/Grey</material>
@@ -60,4 +68,13 @@
     <maxVel>1.0</maxVel>
     <material>Gazebo/Grey</material>
+  </gazebo>
+  <gazebo reference="laser_holder_link">
+    <mu1>30</mu1>
+    <mu2>30</mu2>
+    <kp>1000000.0</kp>
+    <kd>100.0</kd>
+    <minDepth>0.001</minDepth>
+    <maxVel>1.0</maxVel>
+    <material>Gazebo/Red</material>
   </gazebo>
   <gazebo>
@@ -206,4 +223,36 @@
     </sensor>
   </gazebo>
+    <gazebo reference="urg_link">
+        <sensor name="laser" type="ray">
+        <pose>0 0 0 0 0 0</pose>
+          <ray>
+            <scan>
+              <horizontal>
+                <!-- The URG-04LX-UG01  has  683 steps with 0.35139 Degree resolution -->
+                <resolution>1</resolution>
+                <max_angle>2.0944</max_angle> <!-- 120 Degree -->
+                <min_angle>-2.0944</min_angle> <!-- -120 Degree -->
+                <samples>683</samples>
+              </horizontal>
+            </scan>
+            <range>
+              <min>0.08</min>
+              <max>5</max>
+              <resolution>0.01</resolution>
+            </range>
+          </ray>
+          <plugin name="laser" filename="libgazebo_ros_laser.so" >
+            <!--robotNamespace></robotNamespace-->
+            <topicName>urg_scan</topicName>
+            <frameName>urg_link</frameName>
+          </plugin>
+          <!--
+          <plugin name="laser" filename="libRayPlugin.so" />
+          -->
+          <always_on>1</always_on>
+          <update_rate>30</update_rate>
+          <visualize>true</visualize>
+        </sensor>
+    </gazebo>
 <!--
 <gazebo>

File: tb3kai_description/urdf/turtlebot3_burger.urdf.xacro (robot description, xacro)
@@ -180,4 +180,15 @@
   </link>
   <!-- End of Spin Hokuyo -->
+  <!-- Transmission AX-18A ID 3 -->
+  <transmission name="tran1">
+    <type>transmission_interface/SimpleTransmission</type>
+    <joint name="laser_holder_joint">
+      <hardwareInterface>hardware_interface/EffortJointInterface</hardwareInterface>
+    </joint>
+    <actuator name="ax18a3">
+      <hardwareInterface>hardware_interface/EffortJointInterface</hardwareInterface>
+      <mechanicalReduction>1</mechanicalReduction>
+    </actuator>
+  </transmission>
   <!-- URG Hokuyo -->
   <joint name="holder_urg_joint" type="fixed">
